File: Hardware/Spectacle_Accelerometer_Input_Board.sch (EAGLE design)
At the start: 38 parts, among them J19 FTDI_DEVICE, U1 CY8C4146LQI-S422, U2 3.3V/150mA, U3 ADXL345

Commit message: Review feedback
Parts:
- added FD1, FD2: FIDUCIALUFIDUCIAL, SparkFun-Aesthetics:FIDUCIALUFIDUCIAL
- added LOGO3: OSHW-LOGOS, SparkFun-Aesthetics:OSHW-LOGOS
- added LOGO4: SFE_LOGO_NAME_FLAME.1_INCH, SparkFun-Aesthetics:SFE_LOGO_NAME_FLAME.1_INCH
Connections:
- new net N$1: U1G0.P1.7
- new net N$10: U1G3.P2.1
- new net N$12: U1G3.P2.2
- new net N$13: U1G3.P2.3
- new net N$14: U1G3.P2.5
- new net N$15: U1G3.P2.6
- new net N$16: U1G3.P3.1
- new net N$17: U1G3.P3.0
- new net N$18: U1G2.P4.1
- new net N$19: U1G2.P4.2
- new net N$20: U1G2.P4.3
- new net N$7: U1G0.P1.3
- new net N$8: U1G0.P1.2
- new net N$9: U1G3.P2.0
Other:
- note added: "3.5V < VIN < 9V"
Changed lines of the file:
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@@
 <part name="U$2" library="SparkFun-Connectors" deviceset="AUDIO-JACK3" device=""/>
 <part name="GND5" library="SparkFun-Aesthetics" deviceset="GND" device=""/>
+<part name="LOGO3" library="SparkFun-Aesthetics" deviceset="OSHW-LOGO" device="S"/>
+<part name="LOGO4" library="SparkFun-Aesthetics" deviceset="SFE_LOGO_NAME_FLAME" device=".1_INCH"/>
+<part name="FD1" library="SparkFun-Aesthetics" deviceset="FIDUCIAL" device="UFIDUCIAL"/>
+<part name="FD2" library="SparkFun-Aesthetics" deviceset="FIDUCIAL" device="UFIDUCIAL"/>
 </parts>
 <sheets>
@@
 <text x="88.9" y="86.36" size="3.81" layer="97" font="vector">Power
 Supply</text>
+<text x="17.78" y="116.84" size="1.778" layer="97">3.5V &lt; VIN &lt; 9V</text>
 </plain>
 <instances>
@@
 <instance part="U$2" gate="G$1" x="193.04" y="53.34" rot="MR180"/>
 <instance part="GND5" gate="1" x="200.66" y="43.18"/>
+<instance part="LOGO3" gate="G$1" x="78.74" y="10.16"/>
+<instance part="LOGO4" gate="G$1" x="91.44" y="0"/>
+<instance part="FD1" gate="G$1" x="238.76" y="30.48"/>
+<instance part="FD2" gate="G$1" x="241.3" y="30.48"/>
 </instances>
 <busses>
@@
 </segment>
 </net>
+<net name="N$1" class="0">
+<segment>
+<pinref part="U1" gate="G0" pin="P1.7"/>
+<wire x1="152.4" y1="160.02" x2="154.94" y2="160.02" width="0.1524" layer="91"/>
+</segment>
+</net>
+<net name="N$7" class="0">
+<segment>
+<pinref part="U1" gate="G0" pin="P1.3"/>
+<wire x1="152.4" y1="170.18" x2="154.94" y2="170.18" width="0.1524" layer="91"/>
+</segment>
+</net>
+<net name="N$8" class="0">
+<segment>
+<pinref part="U1" gate="G0" pin="P1.2"/>
+<wire x1="152.4" y1="172.72" x2="154.94" y2="172.72" width="0.1524" layer="91"/>
+</segment>
+</net>
+<net name="N$9" class="0">
+<segment>
+<pinref part="U1" gate="G3" pin="P2.0"/>
+<wire x1="167.64" y1="177.8" x2="165.1" y2="177.8" width="0.1524" layer="91"/>
+</segment>
+</net>
+<net name="N$10" class="0">
+<segment>
+<pinref part="U1" gate="G3" pin="P2.1"/>
+<wire x1="167.64" y1="175.26" x2="165.1" y2="175.26" width="0.1524" layer="91"/>
+</segment>
+</net>
+<net name="N$12" class="0">
+<segment>
+<pinref part="U1" gate="G3" pin="P2.2"/>
+<wire x1="167.64" y1="172.72" x2="165.1" y2="172.72" width="0.1524" layer="91"/>
+</segment>
+</net>
+<net name="N$13" class="0">
+<segment>
+<pinref part="U1" gate="G3" pin="P2.3"/>
+<wire x1="167.64" y1="170.18" x2="165.1" y2="170.18" width="0.1524" layer="91"/>
+</segment>
+</net>
+<net name="N$14" class="0">
+<segment>
+<pinref part="U1" gate="G3" pin="P2.5"/>
+<wire x1="167.64" y1="165.1" x2="165.1" y2="165.1" width="0.1524" layer="91"/>
+</segment>
+</net>
+<net name="N$15" class="0">
+<segment>
+<pinref part="U1" gate="G3" pin="P2.6"/>
+<wire x1="167.64" y1="162.56" x2="165.1" y2="162.56" width="0.1524" layer="91"/>
+</segment>
+</net>
+<net name="N$16" class="0">
+<segment>
+<pinref part="U1" gate="G3" pin="P3.1"/>
+<wire x1="195.58" y1="175.26" x2="198.12" y2="175.26" width="0.1524" layer="91"/>
+</segment>
+</net>
+<net name="N$17" class="0">
+<segment>
+<pinref part="U1" gate="G3" pin="P3.0"/>
+<wire x1="195.58" y1="177.8" x2="198.12" y2="177.8" width="0.1524" layer="91"/>
+</segment>
+</net>
+<net name="N$18" class="0">
+<segment>
+<pinref part="U1" gate="G2" pin="P4.1"/>
+<wire x1="152.4" y1="147.32" x2="154.94" y2="147.32" width="0.1524" layer="91"/>
+</segment>
+</net>
+<net name="N$19" class="0">
+<segment>
+<pinref part="U1" gate="G2" pin="P4.2"/>
+<wire x1="152.4" y1="144.78" x2="154.94" y2="144.78" width="0.1524" layer="91"/>
+</segment>
+</net>
+<net name="N$20" class="0">
+<segment>
+<pinref part="U1" gate="G2" pin="P4.3"/>
+<wire x1="152.4" y1="142.24" x2="154.94" y2="142.24" width="0.1524" layer="91"/>
+</segment>
+</net>

Commit message: Fixed issues from Eric's review
Parts:
- D3: value RED -> Yellow; device SparkFun-LED:LED-RED0603 -> SparkFun-LED:LED-YELLOW0603-SMART
Changed lines of the file:
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@@
 <part name="SW1" library="SparkFun-Electromechanical" deviceset="SWITCH_SPST_4_PIN" device="RECT"/>
 <part name="SW2" library="SparkFun-Electromechanical" deviceset="SWITCH_SPST_4_PIN" device="RECT"/>
-<part name="D3" library="SparkFun-LED" deviceset="LED-RED" device="0603" value="RED"/>
+<part name="D3" library="SparkFun-LED" deviceset="LED-YELLOW" device="0603-SMART" value="Yellow"/>
 <part name="R5" library="SparkFun-Resistors" deviceset="1KOHM-1/10W-1%(0603)" device="" value="1K"/>
 <part name="GND12" library="SparkFun-Aesthetics" deviceset="GND" device=""/>

Commit message: Added downstream power control circuitry
Parts:
- added Q1: (no value), SparkFun-DiscreteSemi:IRF7509
- added R10, R11: 10K, SparkFun-Resistors:10KOHM-1/10W-1%(0603)0603
- renumbered J18 to J1, J19 to J2, U$1 to J3, U$2 to J4
Connections:
- removed net N$13: U1G3.P2.3
- new net N$37: Q1NMOS.D, Q1PMOS.G, R11.1
- new net VOUT: D5.2, J4.EARTH, Q1PMOS.D
- new net V_OUT_EN: Q1NMOS.G, R10.1, U1G3.P2.3
- net GND: now also Q1NMOS.S, R10.2
- net VIN: now also D5.1, Q1PMOS.S, R11.2; no longer D5.2, J4.EARTH
Other:
- moved on the sheet: R7, R8, R9, U1G3, U3

Commit message: Added notes to IN and OUT connectors
Other:
- note added: "02"
- note added: "In"
- note added: "Out"
- note removed: "01"
Changed lines of the file:
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@@
 near U3.1</text>
 <text x="167.64" y="7.62" size="3.81" layer="91" font="vector">Mike Hord</text>
-<text x="238.506" y="6.604" size="3.81" layer="91" font="vector">01</text>
+<text x="238.506" y="6.604" size="3.81" layer="91" font="vector">02</text>
 <wire x1="0" y1="83.82" x2="109.22" y2="83.82" width="0.3048" layer="97" style="longdash"/>
 <wire x1="109.22" y1="83.82" x2="147.32" y2="83.82" width="0.3048" layer="97" style="longdash"/>
@@
 Supply</text>
 <text x="17.78" y="116.84" size="1.778" layer="97">3.5V &lt; VIN &lt; 9V</text>
+<text x="184.15" y="73.66" size="1.778" layer="97">In</text>
+<text x="182.372" y="48.26" size="1.778" layer="97">Out</text>
 </plain>
 <instances>
